File: usbDac.sch (EAGLE design)
At the start: 3 parts

Commit message: basic routing
Parts:
- added C10, C11: 100uF, SparkFun-Capacitors:CAP_POLC
- added C3, C4, C5, C8, C9: 1uF, SparkFun-Capacitors:CAP0603-CAP
- added C6, C7: (no value), SparkFun-Capacitors:CAP0603-CAP
- added Q1: (no value), adafruit:XTAL-4-3225
- added R1, R2: 22, SparkFun-Passives:RESISTOR0603-RES
- added R10, R11, R8, R9: 3k3, SparkFun-Passives:RESISTOR0603-RES
- added R3, R4: 1k5, SparkFun-Passives:RESISTOR0603-RES
- added R5: 1M, SparkFun-Passives:RESISTOR0603-RES
- added R6, R7: 16, SparkFun-Passives:RESISTOR0603-RES
- added U1: (no value), SparkFun-Connectors:AUDIO-JACKSMD2
- added X1: USBPCB, SparkFun:USBPCB
Connections:
- new net MUTE: IC1.HID0
- new net N$1: C3.1, IC1.VCCR
- new net N$10: C7.2, IC1.XTO, Q1.X2, R5.1
- new net N$11: IC1.DATA, R4.1
- new net N$12: C10.+, C9.1, IC1.VOUTR, R9.2
- new net N$13: C6.1, Q1.G1
- new net N$14: C11.+, C8.1, IC1.VOUTL, R8.2
- new net N$15: C6.2, IC1.XTI, Q1.X1, R5.2
- new net N$16: C8.2, R6.2
- new net N$17: C9.2, R7.2
- new net N$18: C11.-, R10.2, U1.LEFT
- new net N$19: C10.-, R11.2, U1.RIGHT
- new net N$4: C4.2, IC1.VCCL
- new net N$5: IC1.VBUS, X1.VBUS
- new net N$6: IC1.D+, R1.1
- new net N$7: IC1.D-, R2.1
- new net N$8: R1.2, R3.1, X1.D+
- new net N$9: R2.2, X1.D-
- new net PLAY: IC1.FUNC0
- new net VDD: C5.1, IC1.FSEL, IC1.PSEL, IC1.TEST, IC1.VDD, R3.2, R4.2
- new net VDN: IC1.HID2
- new net VUP: IC1.HID1
- net GND: now also C3.2, C4.1, C5.2, C7.1, IC1.AGNDR, Q1.G2, R10.1, R11.1, R6.1, R7.1, R8.1, R9.1, U1.SLEEVE, X1.GND
Other:
- moved on the sheet: C2

Commit message: routed
Parts:
- C1, C3, C4, C5, C6, C7, C8, C9: device SparkFun-Capacitors:CAP0603-CAP -> SparkFun-Capacitors:CAP0402-CAP
- C10, C11: device SparkFun-Capacitors:CAP_POLC -> SparkFun-Capacitors:CAP_POL6032
- R1, R10, R11, R2, R3, R4, R5, R6, R7, R8, R9: device SparkFun-Passives:RESISTOR0603-RES -> SparkFun-Passives:RESISTOR0402-RES
Connections:
- net N$5 renamed VCC
Changed lines of the file:
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@@
 <part name="IC1" library="PCM2706" deviceset="PCM2706" device=""/>
 <part name="GND1" library="SparkFun-Aesthetics" deviceset="GND" device=""/>
-<part name="C1" library="SparkFun-Capacitors" deviceset="CAP" device="0603-CAP" value="1uF"/>
+<part name="C1" library="SparkFun-Capacitors" deviceset="CAP" device="0402-CAP" value="1uF"/>
 <part name="C2" library="SparkFun-Capacitors" deviceset="CAP_POL" device="1206" value="10uF"/>
-<part name="C3" library="SparkFun-Capacitors" deviceset="CAP" device="0603-CAP" value="1uF"/>
-<part name="C4" library="SparkFun-Capacitors" deviceset="CAP" device="0603-CAP" value="1uF"/>
+<part name="C3" library="SparkFun-Capacitors" deviceset="CAP" device="0402-CAP" value="1uF"/>
+<part name="C4" library="SparkFun-Capacitors" deviceset="CAP" device="0402-CAP" value="1uF"/>
 <part name="X1" library="SparkFun" deviceset="USB" device="PCB"/>
-<part name="R1" library="SparkFun-Passives" deviceset="RESISTOR" device="0603-RES" value="22"/>
-<part name="R2" library="SparkFun-Passives" deviceset="RESISTOR" device="0603-RES" value="22"/>
-<part name="R3" library="SparkFun-Passives" deviceset="RESISTOR" device="0603-RES" value="1k5"/>
-<part name="C5" library="SparkFun-Capacitors" deviceset="CAP" device="0603-CAP" value="1uF"/>
-<part name="R4" library="SparkFun-Passives" deviceset="RESISTOR" device="0603-RES" value="1k5"/>
+<part name="R1" library="SparkFun-Passives" deviceset="RESISTOR" device="0402-RES" value="22"/>
+<part name="R2" library="SparkFun-Passives" deviceset="RESISTOR" device="0402-RES" value="22"/>
+<part name="R3" library="SparkFun-Passives" deviceset="RESISTOR" device="0402-RES" value="1k5"/>
+<part name="C5" library="SparkFun-Capacitors" deviceset="CAP" device="0402-CAP" value="1uF"/>
+<part name="R4" library="SparkFun-Passives" deviceset="RESISTOR" device="0402-RES" value="1k5"/>
 <part name="Q1" library="adafruit" deviceset="XTAL-4" device="-3225"/>
-<part name="C6" library="SparkFun-Capacitors" deviceset="CAP" device="0603-CAP"/>
-<part name="C7" library="SparkFun-Capacitors" deviceset="CAP" device="0603-CAP"/>
-<part name="R5" library="SparkFun-Passives" deviceset="RESISTOR" device="0603-RES" value="1M"/>
-<part name="C8" library="SparkFun-Capacitors" deviceset="CAP" device="0603-CAP" value="1uF"/>
-<part name="C9" library="SparkFun-Capacitors" deviceset="CAP" device="0603-CAP" value="1uF"/>
-<part name="R6" library="SparkFun-Passives" deviceset="RESISTOR" device="0603-RES" value="16"/>
-<part name="R7" library="SparkFun-Passives" deviceset="RESISTOR" device="0603-RES" value="16"/>
-<part name="R8" library="SparkFun-Passives" deviceset="RESISTOR" device="0603-RES" value="3k3"/>
-<part name="R9" library="SparkFun-Passives" deviceset="RESISTOR" device="0603-RES" value="3k3"/>
+<part name="C6" library="SparkFun-Capacitors" deviceset="CAP" device="0402-CAP"/>
+<part name="C7" library="SparkFun-Capacitors" deviceset="CAP" device="0402-CAP"/>
+<part name="R5" library="SparkFun-Passives" deviceset="RESISTOR" device="0402-RES" value="1M"/>
+<part name="C8" library="SparkFun-Capacitors" deviceset="CAP" device="0402-CAP" value="1uF"/>
+<part name="C9" library="SparkFun-Capacitors" deviceset="CAP" device="0402-CAP" value="1uF"/>
+<part name="R6" library="SparkFun-Passives" deviceset="RESISTOR" device="0402-RES" value="16"/>
+<part name="R7" library="SparkFun-Passives" deviceset="RESISTOR" device="0402-RES" value="16"/>
+<part name="R8" library="SparkFun-Passives" deviceset="RESISTOR" device="0402-RES" value="3k3"/>
+<part name="R9" library="SparkFun-Passives" deviceset="RESISTOR" device="0402-RES" value="3k3"/>
 <part name="GND2" library="SparkFun-Aesthetics" deviceset="GND" device=""/>
-<part name="C10" library="SparkFun-Capacitors" deviceset="CAP_POL" device="C" value="100uF"/>
-<part name="C11" library="SparkFun-Capacitors" deviceset="CAP_POL" device="C" value="100uF"/>
-<part name="R10" library="SparkFun-Passives" deviceset="RESISTOR" device="0603-RES" value="3k3"/>
-<part name="R11" library="SparkFun-Passives" deviceset="RESISTOR" device="0603-RES" value="3k3"/>
+<part name="C10" library="SparkFun-Capacitors" deviceset="CAP_POL" device="6032" value="100uF"/>
+<part name="C11" library="SparkFun-Capacitors" deviceset="CAP_POL" device="6032" value="100uF"/>
+<part name="R10" library="SparkFun-Passives" deviceset="RESISTOR" device="0402-RES" value="3k3"/>
+<part name="R11" library="SparkFun-Passives" deviceset="RESISTOR" device="0402-RES" value="3k3"/>
 <part name="U1" library="SparkFun-Connectors" deviceset="AUDIO-JACK" device="SMD2"/>
 </parts>
@@
 </segment>
 </net>
-<net name="N$5" class="0">
+<net name="VCC" class="0">
 <segment>
 <pinref part="IC1" gate="2706" pin="VBUS"/>
@@
 <wire x1="15.24" y1="38.1" x2="15.24" y2="35.56" width="0.1524" layer="91"/>
 <label x="15.24" y="35.56" size="1.016" layer="95" rot="R270" xref="yes"/>
-</segment>
-<segment>
+<junction x="15.24" y="38.1"/>
+</segment>
+<segment>
